Commit message: Add Intel RealSense D435i support for visual SLAM
- Add realsense.yaml config for D435i camera (RGB-D + IMU)
- Add rtabmap.yaml config for visual SLAM with RGB-D
- Add realsense_slam.launch.py with mapping/localization modes
- Update URDF with D435i frames (depth, color, optical)
- Update Dockerfile with librealsense SDK and realsense-ros wrapper
- Update entrypoint to source realsense_ros workspace
- Update README with D435i hardware and roadmap updates

The D435i replaces the Pi Camera and ultrasonic sensor, providing
depth perception for obstacle detection and SLAM.

🤖 Generated with [Claude Code](https://claude.com/claude-code)

Co-Authored-By: Claude Opus 4.5 <noreply@anthropic.com>

File: ros2_ws/src/hexapod_bringup/urdf/hexapod.urdf (robot description, URDF)
Before this commit: robot hexapod, 9 links, 8 joints
Links:
- removed link camera_optical_frame
- added link camera_color_frame
- added link camera_color_optical_frame
- added link camera_depth_frame
- added link camera_depth_optical_frame
- added link camera_imu_optical_frame
- link camera_link: geometry collision box size=0.025 0.090 0.025; visual box size=0.025 0.090 0.025
Joints:
- removed joint camera_optical_joint
- added joint camera_color_joint: type fixed, parent camera_link, child camera_color_frame, origin xyz=0 -0.0175 0 rpy=0 0 0
- added joint camera_color_optical_joint: type fixed, parent camera_color_frame, child camera_color_optical_frame, origin xyz=0 0 0 rpy=-1.5708 0 -1.5708
- added joint camera_depth_joint: type fixed, parent camera_link, child camera_depth_frame, origin xyz=0 0.0175 0 rpy=0 0 0
- added joint camera_depth_optical_joint: type fixed, parent camera_depth_frame, child camera_depth_optical_frame, origin xyz=0 0 0 rpy=-1.5708 0 -1.5708
- added joint camera_imu_joint: type fixed, parent camera_link, child camera_imu_optical_frame, origin xyz=0 0 0 rpy=0 0 0
- joint camera_joint: origin xyz=0.02 0 0.01 rpy=0 0 0 -> xyz=0.03 0 0.01 rpy=0 0 0
- joint ultrasonic_joint: origin xyz=0.03 0 0 rpy=0 0 0 -> xyz=0 0 0 rpy=0 0 0; parent head_tilt_link -> camera_depth_frame
